Commit message: URDF and RVIZ update

File: alpha_sci_description/urdf/base.urdf.xacro (robot description, xacro)
@@ -3,5 +3,5 @@
     <link name="base_link">
         <visual>
-            <origin xyz="0.0 0.0 0.0" rpy="0.0 0.0 0.0"/>
+            <origin xyz="0.2 -0.6 -0.5" rpy="0.0 0.0 1.57079"/>
             <geometry>
                 <mesh filename="package://alpha_sci_description/mesh/alpha_sci.stl" scale="0.001 0.001 0.001"/>
